File: hardware/wildfire-node-v1/wildfire-node-v1-rev-c.kicad_sch (KiCad schematic)
At the start: 30 parts, among them J1 BATT IN (JST-PH 2.0mm 2-pin P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, Q7 TBD, U1 Heltec HTIT-WB32LAF V4.2, U2 PMS5003, U3 AS3935 (SparkFun SEN-15441), U4 BME680, U5 MiniBoost 5V (TPS61023)

Commit message: 0079: A1 3-pin series gate + J2 panel input + full 42-pin Heltec pinout on Rev C
Parts:
- added J2: PANEL IN (13W 5V panel), symbol Connector_Generic:Conn_01x02
Connections:
- net GND: now also A1.3 (GND), J2.2 (Pin_2); no longer A1.2 (GND)
- net at U1.3 (SOLAR): now also A1.2 (SOLAR_OUT); no longer A1.1 (SOLAR_OUT)
- new net SOLAR_IN: A1.1 (SOLAR_IN), J2.1 (Pin_1)
- no-connect marks 7 -> 35
Other:
- note added: "A1 is a 3-pin series gate: J2 PANEL IN -> A1 SOLAR_IN/SOLAR_OUT -> Heltec SOLAR, GND to the star."
- note added: "U1 pins 1-14 keep their 0076/0077 sites (frozen nets); pins 15-42 are added, all NC-flagged."
